File: Node_hw/Node.sch (KiCad schematic (older format))
At the start: 45 parts, among them SW1 SWITCH, SW2 BUTTON, SW3 BUTTON, SW4 BUTTON

Commit message: * CPU & CC1101 changed
Parts:
- removed C11, C22, C7, C8, C9: 0.1u, symbol C
- removed C13: 1u, symbol C
- removed C20, C21: 10pF, CAP_0402, symbol C
- removed DD1: STM32F10X-48, symbol STM32F10X-48
- removed DD?: CC1101, ~, symbol CC1101
- removed R5: 1k, symbol R
- removed R7: 56k, symbol R
- removed TP1: TESTPOINT, symbol TESTPOINT
- removed XL6: CONN_3, symbol CONN_3
- removed XTAL1: 27MHz, 03225, symbol CRYSTAL_H
- added ANT?: ANT_PCB_MONO, ~, symbol ANT_PCB_MONO
- added BLN?: 0896BM15A0001, symbol BALUN868JOHANSON
- added C? (x3): 0.1u, CAP_0402, symbol C
- added C?: 1u, CAP_0402, symbol C
- added C?: 10n, CAP_0402, symbol C
- added C?: 10u, CAP_0603, symbol C
- added C? (x2): 10pF, CAP_0402, symbol C
- added C? (x2): 220pF, symbol C
- added C? (x2): 10n, symbol C
- added C? (x2): 0.1u, symbol C
- added C?: 3.3pF, symbol C
- added C?: 1.8pF, symbol C
- added DD?: CC1101, symbol CC1101
- added DD?: STM32L151CXTX, ~, symbol STM32L151CXTX
- added L?: 5.6nH, IND_0402, symbol L
- added R?: 56k, symbol R
- added R?: 1k, RES_0402, symbol R
- added TP? (x2): TESTPOINT, symbol TESTPOINT
- added XL?: CONN_3, ~, symbol CONN_3
- added XTAL?: 27MHz, 03225, symbol CRYSTAL_H
Connections:
- net labels added: BLUE_LED, CC_GDO2, GREEN_LED, RED_LED, RF1, RF2, UART_RX, UART_TX
- net labels removed: ADC_BAT, Ant1, Ant2, RX1, TX1
- wire segments 127 -> 156
- no-connect marks 17 -> 22
Other:
- note added: "500R07S1R8BV4"
- note added: "CPU"
- note added: "Debug port"
- note added: "L-07C5N6SV4"
- note added: "Matching circuit"
- note added: "Radio"

Commit message: Bottons, LED's and USB were added
Parts:
- added D? (x4): LED, ~, symbol LED
- added XL?: USB_MINI_B, ~, symbol USB_MINI_B
- gave numbers to parts that had none: 1
- renumbered SW2 to SW1, SW3 to SW2, SW4 to SW3
Connections:
- net labels added: BOTTON1, BOTTON2, BOTTON3, BOTTON4, USBDM, USBDP, YELLOW_LED
- wire segments 156 -> 173
- no-connect marks 22 -> 15
Other:
- moved on the sheet: R8, R9, SW1, SW2, SW3, SW4, XL?

Commit message: proceeding
Parts:
- removed R8, R9: 4k7, symbol R
Connections:
- net labels removed: I2C_SCL, I2C_SDA
- wire segments 173 -> 169
Other:
- note added: "Buttons"
- note added: "LEDs"
- moved on the sheet: D?, SW1, SW2, SW3, SW4

Commit message: Добавлен NFC
Parts:
- added C?: 150pF, CAP_0603, symbol C
- added C? (x4): 0.1u, CAP_0603, symbol C
- added C?: 100pF, CAP_0603, symbol C
- added C?: 1u, CAP_0603, symbol C
- added C?: 1n, CAP_0603, symbol C
- added C?: 20pF, CAP_0603, symbol C
- added D?: DIODE, ~, symbol DIODE
- added DA? (x2): GENERIC_8PIN, symbol GENERIC_8PIN
- added L?: 100uH, IND_0402, symbol L
- added Q?: NPN, ~, symbol NPN
- added R2, R? (x4): 1k, RES_0603, symbol R
- added R5, R6, R7, R8: 200, RES_0603, symbol R
- added R?: 20k, RES_0603, symbol R
- added R? (x5): 10k, RES_0603, symbol R
- added R?: 330k, RES_0603, symbol R
- added R?: 100, RES_0603, symbol R
- gave numbers to parts that had none: 32
- renumbered SW1 to SW5
Connections:
- net labels added: +5V, AGND, M_SCL, M_SDA, klNFCModulation, klNFC_Rx, klNFC_Tx, klNFC_Vcc
- net labels removed: BUTTON1, BUTTON2, BUTTON3, BUTTON4
- wire segments 169 -> 244
- no-connect marks 15 -> 12
Other:
- note added: "USB"
- moved on the sheet: B1, C1, C10, C11, C12, C14, C15, C16, C2, C3, C4, C5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

Commit message: * CPU changed to stm32f072 + Simulation * Sch refined
Parts:
- removed DD1: STM32L151CXTX, ~, symbol STM32L151CXTX
- added DD?: STM32F072CXTX, ~, symbol STM32F072CXTX
- DA? (x2): value GENERIC_8PIN -> MAX4453
Connections:
- net labels added: ADC_BATTERY_I, ADC_BATTERY_V, DAC
- net labels removed: M_SCL, M_SDA
- wire segments 244 -> 245
- no-connect marks 12 -> 9
Other:
- moved on the sheet: R1, R2
Changed lines of the file:
@@
 LIBS:Tittar_kl
 LIBS:Transistors_kl
-LIBS:Sensors
 LIBS:display_kl
 LIBS:Antennas_kl
 LIBS:memory
-LIBS:Node-cache
-LIBS:adc_kl
-LIBS:Atmel_kl
-LIBS:Audio_kl
-LIBS:dac
 LIBS:Interface_kl
-LIBS:modules
 LIBS:OpAmp_kl
-LIBS:SmartCard_kl
-LIBS:standard_logic
 LIBS:Node-cache
 EELAYER 27 0
@@
 Sheet 1 1
 Title ""
-Date "8 oct 2014"
+Date "14 nov 2014"
 Rev ""
 Comp ""
@@
 	1    0    0    -1
 $EndComp
-Text Label 5850 2800 0    60   ~ 0
+Text Label 6450 2800 0    60   ~ 0
 SWCLK
-Text Label 5850 2700 0    60   ~ 0
+Text Label 6450 2700 0    60   ~ 0
 SWDIO
 $Comp
 L GND #PWR029
 U 1 1 542517FF
-P 4350 4300
-F 0 "#PWR029" H 4440 4280 30  0001 C CNN
-F 1 "GND" H 4350 4220 30  0001 C CNN
-F 2 "" H 4350 4300 60  0001 C CNN
-F 3 "" H 4350 4300 60  0001 C CNN
-	1    4350 4300
+P 4500 4300
+F 0 "#PWR029" H 4590 4280 30  0001 C CNN
+F 1 "GND" H 4500 4220 30  0001 C CNN
+F 2 "" H 4500 4300 60  0001 C CNN
+F 3 "" H 4500 4300 60  0001 C CNN
+	1    4500 4300
 	1    0    0    -1
 $EndComp
@@
 $EndComp
 NoConn ~ 3100 3100
-Text Label 5850 2300 0    60   ~ 0
+Text Label 6450 2300 0    60   ~ 0
 UART_TX
 $Comp
@@
 Text Notes 13250 2150 0    60   ~ 0
 Matching circuit
-Text Label 5850 1600 0    60   ~ 0
+Text Label 2600 1700 0    60   ~ 0
 CC_GDO2
-Text Label 5850 1700 0    60   ~ 0
+Text Label 2600 1600 0    60   ~ 0
 CC_GDO0
-Text Label 5850 1800 0    60   ~ 0
+Text Label 6450 2200 0    60   ~ 0
 CC_CS
-Text Label 5850 1900 0    60   ~ 0
+Text Label 6450 1900 0    60   ~ 0
 CC_SCK
-Text Label 5850 2000 0    60   ~ 0
+Text Label 6450 2000 0    60   ~ 0
 CC_MISO
-Text Label 5850 2100 0    60   ~ 0
+Text Label 6450 2100 0    60   ~ 0
 CC_MOSI
 $Comp
 L R R1
 U 1 1 54251932
-P 6650 1400
-F 0 "R1" V 6730 1250 50  0000 C CNN
-F 1 "1k" V 6650 1400 50  0000 C CNN
-F 2 "RES_0402" V 6730 1500 28  0000 C CNN
-F 3 "" H 6650 1400 60  0001 C CNN
-	1    6650 1400
+P 7250 1400
+F 0 "R1" V 7330 1250 50  0000 C CNN
+F 1 "1k" V 7250 1400 50  0000 C CNN
+F 2 "RES_0402" V 7330 1500 28  0000 C CNN
+F 3 "" H 7250 1400 60  0001 C CNN
+	1    7250 1400
 	0    -1   -1   0
 $EndComp
@@
 L +BATT #PWR057
 U 1 1 54251938
-P 7000 1400
-F 0 "#PWR057" H 7000 1360 30  0001 C CNN
-F 1 "+BATT" H 7080 1430 30  0000 C CNN
-F 2 "" H 7000 1400 60  0000 C CNN
-F 3 "" H 7000 1400 60  0000 C CNN
-	1    7000 1400
+P 7600 1400
+F 0 "#PWR057" H 7600 1360 30  0001 C CNN
+F 1 "+BATT" H 7680 1430 30  0000 C CNN
+F 2 "" H 7600 1400 60  0000 C CNN
+F 3 "" H 7600 1400 60  0000 C CNN
+	1    7600 1400
 	1    0    0    -1
 $EndComp
@@
 Text Notes 13800 3300 0    60   ~ 0
 500R07S1R8BV4
-Text Label 5850 2400 0    60   ~ 0
+Text Label 6450 2400 0    60   ~ 0
 UART_RX
-NoConn ~ 5750 2200
 $Comp
 L GND #PWR059
@@
 	1    0    0    -1
 $EndComp
-NoConn ~ 5750 3150
-NoConn ~ 5750 3050
-NoConn ~ 5750 2900
+NoConn ~ 6350 3150
+NoConn ~ 6350 3050
 Text Notes 14000 7800 0    60   Italic 12
 Debug port
@@
 Text Label 2950 2200 2    60   ~ 0
 YELLOW_LED
-$Comp
-L STM32L151CXTX DD1
-U 1 1 542519DB
-P 4400 2600
-F 0 "DD1" H 3900 3950 60  0000 C CNN
-F 1 "STM32L151CXTX" H 4550 3950 60  0000 C CNN
-F 2 "~" H 4400 2600 60  0000 C CNN
-F 3 "~" H 4400 2600 60  0000 C CNN
-	1    4400 2600
-	1    0    0    -1
-$EndComp
 Text Label 2950 2600 2    60   ~ 0
 BOTTON1
@@
 	1    0    0    -1
 $EndComp
-Text Label 5850 2500 0    60   ~ 0
+Text Label 6450 2500 0    60   ~ 0
 USBDM
-Text Label 5850 2600 0    60   ~ 0
+Text Label 6450 2600 0    60   ~ 0
 USBDP
 Text Label 15650 9050 0    60   ~ 0
@@
 	0    -1   -1   0
 $EndComp
-Text Label 2950 2400 2    60   ~ 0
-M_SCL
-Text Label 2950 2500 2    60   ~ 0
-M_SDA
 Text Notes 15250 8550 0    60   ~ 12
 USB
@@
 L R R2
 U 1 1 542E3AA1
-P 6650 1600
-F 0 "R2" V 6730 1450 50  0000 C CNN
-F 1 "1k" V 6650 1600 50  0000 C CNN
-F 2 "RES_0603" V 6730 1700 28  0000 C CNN
-F 3 "~" H 6650 1600 60  0000 C CNN
-	1    6650 1600
+P 2100 2000
+F 0 "R2" V 2180 1850 50  0000 C CNN
+F 1 "1k" V 2100 2000 50  0000 C CNN
+F 2 "RES_0603" V 2180 2100 28  0000 C CNN
+F 3 "~" H 2100 2000 60  0000 C CNN
+	1    2100 2000
 	0    -1   -1   0
 $EndComp
@@
 L +5V #PWR069
 U 1 1 542E3C99
-P 7000 1600
-F 0 "#PWR069" H 7000 1560 30  0001 C CNN
-F 1 "+5V" H 7080 1630 30  0000 C CNN
-F 2 "~" H 7000 1600 60  0000 C CNN
-F 3 "~" H 7000 1600 60  0000 C CNN
-	1    7000 1600
-	1    0    0    -1
-$EndComp
-NoConn ~ 3100 1400
-Text Label 2950 2000 2    60   ~ 0
+P 1750 2000
+F 0 "#PWR069" H 1750 1960 30  0001 C CNN
+F 1 "+5V" H 1830 2030 30  0000 C CNN
+F 2 "~" H 1750 2000 60  0000 C CNN
+F 3 "~" H 1750 2000 60  0000 C CNN
+	1    1750 2000
+	-1   0    0    -1
+$EndComp
+Text Label 6800 1500 2    60   ~ 0
 klNFC_Tx
-Text Label 2950 2100 2    60   ~ 0
+Text Label 6800 1700 2    60   ~ 0
 klNFC_Rx
-Text Label 2950 1700 2    60   ~ 0
+Text Label 7100 1600 2    60   ~ 0
 klNFCModulation
 $Comp
@@
 P 2300 9500
 F 0 "DA?" H 2350 9700 60  0000 C CNN
-F 1 "GENERIC_8PIN" H 2500 9800 50  0000 C CNN
+F 1 "MAX4453" H 2500 9800 50  0000 C CNN
 F 2 "" H 2300 9500 60  0000 C CNN
 F 3 "" H 2300 9500 60  0000 C CNN
@@
 P 4350 9500
 F 0 "DA?" H 4400 9700 60  0000 C CNN
-F 1 "GENERIC_8PIN" H 4550 9800 50  0000 C CNN
+F 1 "MAX4453" H 4550 9800 50  0000 C CNN
 F 2 "" H 4350 9500 60  0000 C CNN
 F 3 "" H 4350 9500 60  0000 C CNN
@@
 	6600 5700 6350 5700
 Wire Wire Line
-	6350 6550 6350 5700
+	6350 5700 6350 6550
 Connection ~ 6350 6550
 Wire Wire Line
@@
 	14550 3350 14550 3400
 Wire Wire Line
-	7000 1400 6900 1400
-Wire Wire Line
-	5750 1400 6400 1400
-Wire Wire Line
-	5850 1700 5750 1700
-Wire Wire Line
-	5750 1800 5850 1800
-Wire Wire Line
-	5850 1900 5750 1900
-Wire Wire Line
-	5750 2000 5850 2000
-Wire Wire Line
-	5850 2100 5750 2100
-Wire Wire Line
-	5750 1600 5850 1600
+	7600 1400 7500 1400
+Wire Wire Line
+	6350 1400 7000 1400
+Wire Wire Line
+	6350 2200 6450 2200
+Wire Wire Line
+	6450 1900 6350 1900
+Wire Wire Line
+	6350 2000 6450 2000
+Wire Wire Line
+	6450 2100 6350 2100
 Wire Wire Line
 	13050 2650 11600 2650
@@
 Connection ~ 1950 3250
 Wire Wire Line
-	4350 4050 4350 4300
-Wire Wire Line
-	4150 4050 4150 4150
-Wire Wire Line
-	4150 4150 4600 4150
-Connection ~ 4350 4150
-Wire Wire Line
-	4250 4050 4250 4150
-Connection ~ 4250 4150
-Wire Wire Line
-	4450 4150 4450 4050
+	4500 4050 4500 4300
+Wire Wire Line
+	4300 4050 4300 4150
+Wire Wire Line
+	4300 4150 4750 4150
+Connection ~ 4500 4150
+Wire Wire Line
+	4400 4050 4400 4150
+Connection ~ 4400 4150
 Wire Wire Line
 	4600 4150 4600 4050
-Connection ~ 4450 4150
+Wire Wire Line
+	4750 4150 4750 4050
+Connection ~ 4600 4150
 Wire Wire Line
 	2400 3450 3100 3450
@@
 Wire Wire Line
 	11150 7100 11000 7100
-Wire Wire Line
-	3100 2400 2950 2400
-Wire Wire Line
-	3100 2500 2950 2500
 Wire Notes Line
 	8250 11200 8350 11200
 Wire Wire Line
-	5750 2300 5850 2300
-Wire Wire Line
-	5750 2400 5850 2400
-Wire Wire Line
-	5750 2500 5850 2500
-Wire Wire Line
-	5750 2600 5850 2600
-Wire Wire Line
-	5750 2700 5850 2700
-Wire Wire Line
-	5750 2800 5850 2800
-Wire Wire Line
-	5750 1500 6400 1500
-Wire Wire Line
-	6400 1500 6400 1600
-Wire Wire Line
-	6900 1600 7000 1600
-Wire Wire Line
-	3100 2000 2950 2000
-Wire Wire Line
-	3100 2100 2950 2100
-Wire Wire Line
-	3100 1700 2050 1700
-Wire Wire Line
-	2050 1700 2050 1600
-Wire Wire Line
-	2050 1600 3100 1600
+	6350 2300 6450 2300
+Wire Wire Line
+	6350 2400 6450 2400
+Wire Wire Line
+	6350 2500 6450 2500
+Wire Wire Line
+	6350 2600 6450 2600
+Wire Wire Line
+	6350 2700 6450 2700
+Wire Wire Line
+	6350 2800 6450 2800
+Wire Wire Line
+	1850 2000 1750 2000
 Wire Wire Line
 	700  10200 700  10300
@@
 	1    0    0    -1
 $EndComp
+Wire Wire Line
+	6800 1500 6350 1500
+Wire Wire Line
+	6350 1700 6800 1700
+Wire Wire Line
+	6350 1600 7100 1600
+Wire Wire Line
+	7100 1600 7100 2900
+Wire Wire Line
+	7100 2900 6350 2900
+Text Label 6500 1800 0    60   ~ 0
+DAC
+Wire Wire Line
+	6500 1800 6350 1800
+Text Label 2350 1400 0    60   ~ 0
+ADC_BATTERY_V
+Text Label 2350 1500 0    60   ~ 0
+ADC_BATTERY_I
+Wire Wire Line
+	2350 1500 3100 1500
+Wire Wire Line
+	3100 1400 2350 1400
+Wire Wire Line
+	2600 1600 3100 1600
+Wire Wire Line
+	3100 1700 2600 1700
+Wire Wire Line
+	2350 2000 3100 2000
+$Comp
+L STM32F072CXTX DD?
+U 1 1 5466687D
+P 4550 2600
+F 0 "DD?" H 4050 3950 60  0000 C CNN
+F 1 "STM32F072CXTX" H 4700 3950 60  0000 C CNN
+F 2 "~" H 4550 2600 60  0000 C CNN
+F 3 "~" H 4550 2600 60  0000 C CNN
+	1    4550 2600
+	1    0    0    -1
+$EndComp
+Text Label 2500 2400 0    60   ~ 0
+klNFC_Vcc
+Wire Wire Line
+	2500 2400 3100 2400
 $EndSCHEMATC
